File: CAD/kicad/Starbie.kicad_pcb (KiCad board)
At the start: 2 copper layers, 152.4 x 139.7 mm, 7 parts, among them J1 Conn_01x04_Pin, J2 Conn_01x08_Pin, SW1 SW_Push, SW2 SW_Push, U1 XIAO-ESP32-C3-SMD, U2 DHT11

Commit message: see journal.md
Parts:
- added D1: D_Schottky, Diode_THT:D_DO-41_SOD81_P7.62mm_Horizontal, F.Cu at (161.9, 79.0)
- added F1: Polyfuse, Fuse:Fuse_1812_4532Metric, F.Cu at (163.9, 144.1)
- added J3: Conn_01x02, Battery:BatteryHolder_TruPower_BH-331P_3xAA, B.Cu at (152.6, 86.6)
- added R2: 100k, Resistor_THT:R_Axial_DIN0204_L3.6mm_D1.6mm_P7.62mm_Horizontal, F.Cu at (174.9, 78.7)
- added R3: 47k, Resistor_THT:R_Axial_DIN0204_L3.6mm_D1.6mm_P7.62mm_Horizontal, F.Cu at (186.9, 78.2)
- added SW3: SW_SPDT, Connector_PinHeader_2.54mm:PinHeader_1x03_P2.54mm_Vertical, F.Cu at (173.5, 94.2)
- moved R1 4.00 mm to (111.5, 93.4)
- moved J1 3.83 mm to (127.1, 59.5)
- moved SW1 1.47 mm to (100.5, 83.8)
Connections:
- U1 pad 1: unconnected-(U1-D0-Pad1) -> /BAT_SENSE
Routing:
- net +3.3V: track 127.6 -> 258.9 mm, vias 0 -> 2
- net /DHT11 DATA: track 50.0 -> 159.2 mm, vias 0 -> 2
- net /VBAT: track 0.00 -> 82.0 mm
- net /BAT_SENSE: track 0.00 -> 80.6 mm
- net /SCL: track 91.1 -> 160.0 mm
- net /SDA: track 96.5 -> 147.1 mm
- net Net-(SW3-C): track 0.00 -> 49.7 mm
- net +5V: track 0.00 -> 41.4 mm
- net /Battery+: track 0.00 -> 25.8 mm, vias 0 -> 1
- net GND: track 187.1 -> 202.1 mm
- net /Button 1 Net: track 46.3 -> 51.0 mm, vias 0 -> 1

Commit message: Updated Gerbers and cad files with an led
Parts:
- added D2: LED, LED_THT:LED_D5.0mm, F.Cu at (100.2, 134.4)
- added R4: 330, Resistor_THT:R_Axial_DIN0204_L3.6mm_D1.6mm_P7.62mm_Horizontal, F.Cu at (88.5, 132.8)
Connections:
- U1 pad 11: unconnected-(U1-D10-Pad11) -> /LED
Routing:
- net /LED: track 0.00 -> 66.5 mm, vias 0 -> 1
- net GND: track 202.1 -> 236.4 mm, vias 0 -> 1
- net Net-(D2-A): track 0.00 -> 7.28 mm
